File: hardware/quadcopter.sch (EAGLE design)
At the start: 63 parts, among them J1 AVR_SPI_PRG_6NS, J2 HEADER-0.1IN-2POS-MALE, J3 FTDI_BASICPTH, M1 MOTOR_PADS-MOLEX-0530470210, M1HEADER HEADER-0.1IN-3POS, M2 MOTOR_PADS-MOLEX-0530470210, M2HEADER HEADER-0.1IN-3POS, M3 MOTOR_PADS-MOLEX-0530470210, M3HEADER HEADER-0.1IN-3POS, M4 MOTOR_PADS-MOLEX-0530470210, M4HEADER HEADER-0.1IN-3POS, Q1 FET, Q2 FET, Q3 FET, Q4 FET, U1 ATMEGA128RFA1, U2 IMU-LSM, Y1 CRYSTAL5X3

Commit message: Add files via upload
Parts:
- removed BRIDGE, BRIDGE3: NET_BRIDGE, custom:NET_BRIDGE
- removed IMUHEADER, IMURESCUE: HEADER-4POS-0.1IN-FEMALE, quadparts_prebuilt:HEADER-4POS-0.1IN-FEMALE
- removed M1, M2, M3, M4: MOTOR_PADS-MOLEX-0530470210, quadparts_prebuilt:MOTOR_PADS-MOLEX-0530470210
- removed M1HEADER, M2HEADER, M3HEADER, M4HEADER: HEADER-0.1IN-3POS, quadparts_prebuilt:HEADER-0.1IN-3POS
- removed V1: 3.3V, quadparts_prebuilt:TPS73633-DBVT3V3
- added D10, D11, D12, D13, D14, D15, D16, D17, D18, D19, D20, D8: BLUE, LED:DIODE-LED-SMD-2012-0805-BLUE-BLUE
- added D21, D9: red, LED:DIODE-LED-SMD-2012-0805-RED-RED
- added J4: (no value), quadparts_prebuilt:HEADER-10POSTH-254X10
- added J5: HEADER-4POS-0.1IN-FEMALE, quadparts_prebuilt:HEADER-4POS-0.1IN-FEMALE
- added Q5: MOSFET-VISHAY-SOT23-N-MOSFET, custom:MOSFET-VISHAY-SOT23-N-MOSFET
- added R10, R9: 10K, quadparts_prebuilt:RESISTOR_SMD-2012-0805-10K
- added R11, R14, R15, R16, R17, R18, R19, R20, R21, R22, R23, R24: 28, custom:RESISTOR_SMD-2012-0805-28
- added R12, R13, R25, R26, R27, R28: 86.6, custom:RESISTOR_SMD-2012-0805-88.6
- added U$1, U$2, U$3, U$4: yellow, LED:DIODE-LED-SMD-2012-0805-YELLOW-YELLOW
- added U3, U4, U5, U6: MOTOR_PADS-MOLEX-0530470210, quadparts_prebuilt:MOTOR_PADS-MOLEX-0530470210
- added U7: 3.3V, quadparts_prebuilt:TPS73633-DBVT3V3
- added U8: NET_BRIDGE-BRIDGE-SMD, custom:NET_BRIDGE-BRIDGE-SMD
- C12: value 0.1uF -> 0.01uF; device quadparts_prebuilt:CAPACITOR-NP_SMD-2012-0805_CERAMIC-0.1UF -> quadparts_prebuilt:CAPACITOR-NP_SMD-2012-0805_CERAMIC-0.01UF
- C13: value 10uF -> 0.1uF; device quadparts_prebuilt:CAPACITOR-NP_SMD-2012-0805_CERAMIC-10UF -> quadparts_prebuilt:CAPACITOR-NP_SMD-2012-0805_CERAMIC-0.1UF
- D2: device custom:LED-RED -> custom:LED-LITEON-C170EKT-RED-LED
- Q1, Q2, Q3, Q4: value FET -> MOSFET-VISHAY-SOT23-N-MOSFET; device custom:FET -> custom:MOSFET-VISHAY-SOT23-N-MOSFET
- R1: value 330 -> 10K; device quadparts_prebuilt:RESISTOR_SMD-2012-0805-330 -> quadparts_prebuilt:RESISTOR_SMD-2012-0805-10K
- R3: value 10K -> 330; device quadparts_prebuilt:RESISTOR_SMD-2012-0805-10K -> quadparts_prebuilt:RESISTOR_SMD-2012-0805-330
- U2: value IMU-LSM -> IMU_LSM-ST-LSM9DS1-IMU-LGA; device custom:IMU-LSM -> custom:IMU_LSM-ST-LSM9DS1-IMU-LGA
Connections:
- net A8 renamed N$1
- net B1-3 renamed N$4
- net B1-4 renamed N$3
- net C3 renamed N$2
- net C5 renamed N$5
- net C6 renamed N$6
- net C8 renamed N$8
- net C9 renamed N$11
- net CAP renamed N$13
- removed net C1: C10.1, U2.C1
- removed net D1: D1.A, R1.1
- removed net D2: D2.A, R2.1
- removed net PWR: C15.+, C16.+, C17.+, C18.+, D3.C, D4.C, D5.C, D6.C, M1.V+, M2.V+, M3.V+, M4.V+
- removed net Q1: D3.A, M1.V-, Q1.D
- removed net Q2: D4.A, M2.V-, Q2.D
- removed net Q3: D5.A, M3.V-, Q3.D
- removed net Q4: D6.A, M4.V-, Q4.D
- removed net VBAT1: M2HEADER.1
- removed net VBAT2: M3HEADER.1
- removed net VBAT3: M4HEADER.1
- new net N$10: D2.A, R3.1
- new net N$12: C13.1, U2.C1
- new net N$14: D3.A, Q1.D, U3.V-
- new net N$15: B2.P, J2.1
- new net N$16: D4.A, Q2.D, U4.V-
- new net N$17: D21.A, R28.1
- new net N$18: D5.A, Q3.D, U5.V-
- new net N$20: D6.A, Q4.D, U6.V-
- new net N$21: D9.A, R12.1
- new net N$22: R27.1, U$4.A
- new net N$23: R26.1, U$3.A
- new net N$24: R25.1, U$2.A
- new net N$25: R13.1, U$1.A
- new net N$26: D20.A, R24.1
- new net N$27: D19.A, R23.1
- new net N$28: D18.A, R22.1
- new net N$29: D17.A, R21.1
- new net N$30: D16.A, R20.1
- new net N$31: D15.A, R19.1
- new net N$32: D14.A, R18.1
- new net N$33: D13.A, R17.1
- new net N$34: D12.A, R16.1
- new net N$35: D11.A, R15.1
- new net N$36: D10.A, R14.1
- new net N$37: D8.A, R11.1
- new net N$38: D10.C, D11.C, D12.C, D13.C, D14.C, D15.C, D16.C, D17.C, D18.C, D19.C, D20.C, D21.C, D8.C, D9.C, Q5.D, U$1.C, U$2.C, U$3.C, U$4.C
- new net N$9: D1.A, R2.1
- net 3: now also J4.7, Q2.G, R7.2; no longer M1HEADER.2, Q1.G, R3.1
- net 3V3: now also C10.1, J4.6, J5.4, R1.2, R4.2, R5.2, U7.OUT; no longer B3.1, BRIDGE3.2, C13.1, IMUHEADER.4, IMURESCUE.4, J1.2, J3.4, R5.1, R6.1, U1.RSTN, V1.OUT
- net 4: now also J4.8, Q3.G, R8.2; no longer M2HEADER.2, Q2.G, R4.1
- net 5: now also J4.9, Q4.G, R9.2; no longer M3HEADER.2, Q3.G, R7.1
- net 8: now also J4.5, Q1.G, R6.2; no longer M4HEADER.2, Q4.G, R8.1
- net 9: now also Q5.G, R10.2
- net BAT_GND: now also J4.1, Q5.S, U8.P1; no longer BRIDGE.2, C20.2, M1HEADER.3, M2HEADER.3, M3HEADER.3, M4HEADER.3
- net GND: now also C20.2, J4.2, J5.1, R10.1, R6.1, R7.1, R8.1, R9.1, U7.GND, U8.P2; no longer BRIDGE.1, IMUHEADER.1, IMURESCUE.1, R3.2, R4.2, R7.2, R8.2, V1.GND
- net PG0: now also R2.2; no longer R1.2
- net PG1: now also R3.2; no longer R2.2
- net RESET: now also B3.1, R1.1, U1.RSTN
- net SCL: now also J4.3, J5.2, R5.1; no longer IMUHEADER.2, IMURESCUE.2, R6.2
- net SDA: now also J4.4, J5.3, R4.1; no longer IMUHEADER.3, IMURESCUE.3, R5.2
- net VBAT: now also C15.+, C16.+, C17.+, C18.+, D3.C, D4.C, D5.C, D6.C, J4.10, R11.2, R12.2, R13.2, R14.2, R15.2, R16.2, R17.2, R18.2, R19.2, R20.2, R21.2, R22.2, R23.2, R24.2, R25.2, R26.2, R27.2, R28.2, U3.V+, U4.V+, U5.V+, U6.V+; no longer B2.P, C20.1, J2.1, M1HEADER.1, V1.EN
- net VIN: now also C20.1, J1.2, J3.4, U7.EN, U7.IN; no longer BRIDGE3.1, V1.IN
Other:
- note added: "IMU RESCUE"
- note added: "IMU_LSM9DS1"
- note added: "LED CONNECTTIONS"
- note added: "MOTOR DRIVER"
- note added: "SIGNALS"
- note removed: "IMU"
- note removed: "IMU RESCUE HEADER"
- note removed: "Motor 1 Driver"
- note removed: "Motor 2 Driver"
- note removed: "Motor 3 Driver"
- note removed: "Motor 4 Driver"
- moved on the sheet: A8, B1, B2, B3, C1, C10, C11, C12, C13, C14, C15, C16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

Commit message: Add files via upload
Parts:
- renumbered U$1 to D22, U$2 to D23, U$3 to D24, U$4 to D25
Changed lines of the file:
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@@
 <part name="R12" library="custom" deviceset="RESISTOR_" device="SMD-2012-0805-88.6" value="86.6"/>
 <part name="D9" library="LED" deviceset="DIODE-LED-SMD-2012-0805-RED" device="-RED" value="red"/>
-<part name="U$1" library="LED" deviceset="DIODE-LED-SMD-2012-0805-YELLOW" device="-YELLOW" value="yellow"/>
+<part name="D22" library="LED" deviceset="DIODE-LED-SMD-2012-0805-YELLOW" device="-YELLOW" value="yellow"/>
 <part name="R13" library="custom" deviceset="RESISTOR_" device="SMD-2012-0805-88.6" value="86.6"/>
 <part name="D10" library="LED" deviceset="DIODE-LED-SMD-2012-0805-BLUE" device="-BLUE" value="BLUE"/>
@@
 <part name="D20" library="LED" deviceset="DIODE-LED-SMD-2012-0805-BLUE" device="-BLUE" value="BLUE"/>
 <part name="R24" library="custom" deviceset="RESISTOR_" device="SMD-2012-0805-28" value="28"/>
-<part name="U$2" library="LED" deviceset="DIODE-LED-SMD-2012-0805-YELLOW" device="-YELLOW" value="yellow"/>
+<part name="D23" library="LED" deviceset="DIODE-LED-SMD-2012-0805-YELLOW" device="-YELLOW" value="yellow"/>
 <part name="R25" library="custom" deviceset="RESISTOR_" device="SMD-2012-0805-88.6" value="86.6"/>
-<part name="U$3" library="LED" deviceset="DIODE-LED-SMD-2012-0805-YELLOW" device="-YELLOW" value="yellow"/>
+<part name="D24" library="LED" deviceset="DIODE-LED-SMD-2012-0805-YELLOW" device="-YELLOW" value="yellow"/>
 <part name="R26" library="custom" deviceset="RESISTOR_" device="SMD-2012-0805-88.6" value="86.6"/>
-<part name="U$4" library="LED" deviceset="DIODE-LED-SMD-2012-0805-YELLOW" device="-YELLOW" value="yellow"/>
+<part name="D25" library="LED" deviceset="DIODE-LED-SMD-2012-0805-YELLOW" device="-YELLOW" value="yellow"/>
 <part name="R27" library="custom" deviceset="RESISTOR_" device="SMD-2012-0805-88.6" value="86.6"/>
 <part name="R28" library="custom" deviceset="RESISTOR_" device="SMD-2012-0805-88.6" value="86.6"/>
@@
 <attribute name="VALUE" x="365.76" y="-43.18" size="1.778" layer="96" font="vector" rot="MR270"/>
 </instance>
-<instance part="U$1" gate="G$1" x="327.66" y="-45.72" smashed="yes" rot="MR270">
+<instance part="D22" gate="G$1" x="327.66" y="-45.72" smashed="yes" rot="MR270">
 <attribute name="NAME" x="325.12" y="-43.18" size="1.778" layer="95" font="vector" rot="MR270"/>
 <attribute name="VALUE" x="330.2" y="-43.18" size="1.778" layer="96" font="vector" rot="MR270"/>
@@
 <attribute name="NAME" x="313.4614" y="-39.37" size="1.778" layer="95" rot="R90"/>
 </instance>
-<instance part="U$2" gate="G$1" x="335.28" y="-45.72" smashed="yes" rot="MR270">
+<instance part="D23" gate="G$1" x="335.28" y="-45.72" smashed="yes" rot="MR270">
 <attribute name="NAME" x="332.74" y="-43.18" size="1.778" layer="95" font="vector" rot="MR270"/>
 <attribute name="VALUE" x="337.82" y="-43.18" size="1.778" layer="96" font="vector" rot="MR270"/>
@@
 <attribute name="NAME" x="333.7814" y="-39.37" size="1.778" layer="95" rot="R90"/>
 </instance>
-<instance part="U$3" gate="G$1" x="342.9" y="-45.72" smashed="yes" rot="MR270">
+<instance part="D24" gate="G$1" x="342.9" y="-45.72" smashed="yes" rot="MR270">
 <attribute name="NAME" x="340.36" y="-43.18" size="1.778" layer="95" font="vector" rot="MR270"/>
 <attribute name="VALUE" x="345.44" y="-43.18" size="1.778" layer="96" font="vector" rot="MR270"/>
@@
 <attribute name="NAME" x="341.4014" y="-39.37" size="1.778" layer="95" rot="R90"/>
 </instance>
-<instance part="U$4" gate="G$1" x="350.52" y="-45.72" smashed="yes" rot="MR270">
+<instance part="D25" gate="G$1" x="350.52" y="-45.72" smashed="yes" rot="MR270">
 <attribute name="NAME" x="347.98" y="-43.18" size="1.778" layer="95" font="vector" rot="MR270"/>
 <attribute name="VALUE" x="353.06" y="-43.18" size="1.778" layer="96" font="vector" rot="MR270"/>
@@
 <wire x1="187.96" y1="-43.18" x2="187.96" y2="-38.1" width="0.1524" layer="91"/>
 <junction x="187.96" y="-38.1"/>
-</segment>
-<segment>
-<pinref part="J2" gate="G$1" pin="2"/>
-<wire x1="50.8" y1="142.24" x2="50.8" y2="139.7" width="0.1524" layer="91"/>
-<wire x1="50.8" y1="139.7" x2="55.88" y2="139.7" width="0.1524" layer="91"/>
-<pinref part="P+19" gate="VCC" pin="VBAT"/>
-<wire x1="55.88" y1="139.7" x2="55.88" y2="154.94" width="0.1524" layer="91"/>
 </segment>
 <segment>
@@
 <junction x="363.22" y="-30.48"/>
 </segment>
+<segment>
+<pinref part="P+19" gate="VCC" pin="VBAT"/>
+<wire x1="55.88" y1="154.94" x2="55.88" y2="139.7" width="0.1524" layer="91"/>
+<wire x1="55.88" y1="139.7" x2="50.8" y2="139.7" width="0.1524" layer="91"/>
+<pinref part="J2" gate="G$1" pin="2"/>
+<wire x1="50.8" y1="139.7" x2="50.8" y2="142.24" width="0.1524" layer="91"/>
+</segment>
 </net>
 <net name="BAT_GND" class="0">
@@
 <segment>
 <pinref part="R27" gate="G$1" pin="1"/>
-<pinref part="U$4" gate="G$1" pin="A"/>
+<pinref part="D25" gate="G$1" pin="A"/>
 <wire x1="350.52" y1="-40.64" x2="350.52" y2="-43.18" width="0.1524" layer="91"/>
 </segment>
@@
 <segment>
 <pinref part="R26" gate="G$1" pin="1"/>
-<pinref part="U$3" gate="G$1" pin="A"/>
+<pinref part="D24" gate="G$1" pin="A"/>
 <wire x1="342.9" y1="-40.64" x2="342.9" y2="-43.18" width="0.1524" layer="91"/>
 </segment>
@@
 <segment>
 <pinref part="R25" gate="G$1" pin="1"/>
-<pinref part="U$2" gate="G$1" pin="A"/>
+<pinref part="D23" gate="G$1" pin="A"/>
 <wire x1="335.28" y1="-40.64" x2="335.28" y2="-43.18" width="0.1524" layer="91"/>
 </segment>
@@
 <segment>
 <pinref part="R13" gate="G$1" pin="1"/>
-<pinref part="U$1" gate="G$1" pin="A"/>
+<pinref part="D22" gate="G$1" pin="A"/>
 <wire x1="327.66" y1="-40.64" x2="327.66" y2="-43.18" width="0.1524" layer="91"/>
 </segment>
@@
 <wire x1="314.96" y1="-53.34" x2="307.34" y2="-53.34" width="0.1524" layer="91"/>
 <junction x="307.34" y="-53.34"/>
-<pinref part="U$1" gate="G$1" pin="C"/>
+<pinref part="D22" gate="G$1" pin="C"/>
 <wire x1="327.66" y1="-50.8" x2="327.66" y2="-53.34" width="0.1524" layer="91"/>
 <wire x1="327.66" y1="-53.34" x2="314.96" y2="-53.34" width="0.1524" layer="91"/>
 <junction x="314.96" y="-53.34"/>
-<pinref part="U$2" gate="G$1" pin="C"/>
+<pinref part="D23" gate="G$1" pin="C"/>
 <wire x1="335.28" y1="-50.8" x2="335.28" y2="-53.34" width="0.1524" layer="91"/>
 <wire x1="335.28" y1="-53.34" x2="327.66" y2="-53.34" width="0.1524" layer="91"/>
 <junction x="327.66" y="-53.34"/>
-<pinref part="U$3" gate="G$1" pin="C"/>
+<pinref part="D24" gate="G$1" pin="C"/>
 <wire x1="342.9" y1="-50.8" x2="342.9" y2="-53.34" width="0.1524" layer="91"/>
 <wire x1="342.9" y1="-53.34" x2="335.28" y2="-53.34" width="0.1524" layer="91"/>
 <junction x="335.28" y="-53.34"/>
-<pinref part="U$4" gate="G$1" pin="C"/>
+<pinref part="D25" gate="G$1" pin="C"/>
 <wire x1="350.52" y1="-50.8" x2="350.52" y2="-53.34" width="0.1524" layer="91"/>
 <wire x1="350.52" y1="-53.34" x2="342.9" y2="-53.34" width="0.1524" layer="91"/>

Commit message: Add files via upload
Parts:
- D2: device custom:LED-LITEON-C170EKT-RED-LED -> LED:DIODE-LED-LITEON-C170EKT-RED-LITEON-C170EKT-RED-LED
Changed lines of the file:
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@@
 <part name="GND14" library="quadparts_prebuilt" deviceset="GND" device=""/>
 <part name="D1" library="quadparts_prebuilt" deviceset="DIODE-LED_" device="SMD-2012-0805-GREEN" value="green"/>
-<part name="D2" library="custom" deviceset="LED" device="-LITEON-C170EKT-RED-LED" value="red"/>
 <part name="R2" library="quadparts_prebuilt" deviceset="RESISTOR_" device="SMD-2012-0805-330" value="330"/>
 <part name="R3" library="quadparts_prebuilt" deviceset="RESISTOR_" device="SMD-2012-0805-330" value="330"/>
@@
 <part name="R28" library="custom" deviceset="RESISTOR_" device="SMD-2012-0805-88.6" value="86.6"/>
 <part name="D21" library="LED" deviceset="DIODE-LED-SMD-2012-0805-RED" device="-RED" value="red"/>
+<part name="D2" library="LED" deviceset="DIODE-LED-LITEON-C170EKT-RED" device="-LITEON-C170EKT-RED-LED" value="red"/>
 </parts>
 <sheets>
@@
 <attribute name="VALUE" x="182.753" y="104.902" size="1.778" layer="96" rot="R270"/>
 </instance>
-<instance part="D2" gate="G$1" x="198.12" y="99.06" smashed="yes" rot="MR270">
-<attribute name="NAME" x="203.2" y="106.68" size="1.27" layer="95" font="vector" rot="MR270"/>
-<attribute name="VALUE" x="195.58" y="106.68" size="1.27" layer="96" font="vector" rot="MR270"/>
-</instance>
 <instance part="R2" gate="G$1" x="187.96" y="116.84" smashed="yes" rot="R90">
 <attribute name="VALUE" x="191.262" y="113.03" size="1.778" layer="96" rot="R90"/>
@@
 <attribute name="NAME" x="368.3" y="-43.18" size="1.778" layer="95" font="vector" rot="MR270"/>
 <attribute name="VALUE" x="373.38" y="-43.18" size="1.778" layer="96" font="vector" rot="MR270"/>
+</instance>
+<instance part="D2" gate="G$1" x="198.12" y="101.6" smashed="yes" rot="R270">
+<attribute name="NAME" x="200.66" y="104.14" size="1.778" layer="95" font="vector" rot="R270"/>
+<attribute name="VALUE" x="193.04" y="104.14" size="1.778" layer="96" font="vector" rot="R270"/>
 </instance>
 </instances>
@@
 </segment>
 <segment>
-<pinref part="D2" gate="G$1" pin="C"/>
 <pinref part="GND13" gate="1" pin="GND"/>
 <wire x1="198.12" y1="96.52" x2="198.12" y2="93.98" width="0.1524" layer="91"/>
+<pinref part="D2" gate="G$1" pin="C"/>
 </segment>
 <segment>
@@
 <net name="N$10" class="0">
 <segment>
+<pinref part="R3" gate="G$1" pin="1"/>
 <pinref part="D2" gate="G$1" pin="A"/>
-<pinref part="R3" gate="G$1" pin="1"/>
-<wire x1="198.12" y1="109.22" x2="198.12" y2="111.76" width="0.1524" layer="91"/>
-</segment>
-</net>
+<wire x1="198.12" y1="111.76" x2="198.12" y2="104.14" width="0.1524" layer="91"/>
+</segment>
+</net>

Commit message: Add files via upload
Parts:
- removed J4: (no value), quadparts_prebuilt:HEADER-10POSTH-254X10
- added J6: (no value), quadparts_prebuilt:SIP-10_TH-254X10
Connections:
- net 3: now also J6.4; no longer J4.7
- net 3V3: now also J6.5; no longer J4.6
- net 4: now also J6.3; no longer J4.8
- net 5: now also J6.2; no longer J4.9
- net 8: now also J6.6; no longer J4.5
- net BAT_GND: now also J6.10; no longer J4.1
- net GND: now also J6.9; no longer J4.2
- net SCL: now also J6.8; no longer J4.3
- net SDA: now also J6.7; no longer J4.4
- net VBAT: now also J6.1; no longer J4.10
Changed lines of the file:
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@@
 <part name="D7" library="quadparts_prebuilt" deviceset="DIODE-SCHOTTKY_" device="SMD-SOD123-360MV" value="360mV"/>
 <part name="U8" library="custom" deviceset="NET_BRIDGE" device="-BRIDGE-SMD"/>
-<part name="J4" library="quadparts_prebuilt" deviceset="HEADER-10POS" device="TH-254X10"/>
 <part name="P+5" library="quadparts_prebuilt" deviceset="VBAT" device=""/>
 <part name="P+6" library="quadparts_prebuilt" deviceset="3V3" device=""/>
@@
 <part name="D21" library="LED" deviceset="DIODE-LED-SMD-2012-0805-RED" device="-RED" value="red"/>
 <part name="D2" library="LED" deviceset="DIODE-LED-LITEON-C170EKT-RED" device="-LITEON-C170EKT-RED-LED" value="red"/>
+<part name="J6" library="quadparts_prebuilt" deviceset="SIP-10_" device="TH-254X10"/>
 </parts>
 <sheets>
@@
 <attribute name="NAME" x="53.34" y="124.46" size="1.27" layer="95" font="vector"/>
 </instance>
-<instance part="J4" gate="G$1" x="363.22" y="127" smashed="yes" rot="MR0">
-<attribute name="VALUE" x="363.22" y="124.46" size="1.778" layer="96" rot="MR0"/>
-<attribute name="NAME" x="356.362" y="127" size="1.778" layer="95"/>
-</instance>
 <instance part="P+5" gate="VCC" x="345.44" y="157.48" smashed="yes">
 <attribute name="VALUE" x="345.44" y="160.02" size="1.778" layer="96" rot="R180" align="center"/>
@@
 <attribute name="NAME" x="200.66" y="104.14" size="1.778" layer="95" font="vector" rot="R270"/>
 <attribute name="VALUE" x="193.04" y="104.14" size="1.778" layer="96" font="vector" rot="R270"/>
+</instance>
+<instance part="J6" gate="G$1" x="363.22" y="154.94" smashed="yes" rot="R180">
+<attribute name="VALUE" x="363.22" y="157.48" size="1.778" layer="96" rot="R180"/>
+<attribute name="NAME" x="356.362" y="154.94" size="1.778" layer="95" rot="R180"/>
 </instance>
 </instances>
@@
 </segment>
 <segment>
-<pinref part="J4" gate="G$1" pin="5"/>
 <wire x1="353.06" y1="139.7" x2="350.52" y2="139.7" width="0.1524" layer="91"/>
 <label x="350.52" y="139.7" size="1.27" layer="95" font="vector" rot="R180" xref="yes"/>
+<pinref part="J6" gate="G$1" pin="6"/>
 </segment>
 </net>
@@
 </segment>
 <segment>
-<pinref part="J4" gate="G$1" pin="7"/>
 <wire x1="353.06" y1="144.78" x2="350.52" y2="144.78" width="0.1524" layer="91"/>
 <label x="350.52" y="144.78" size="1.27" layer="95" font="vector" rot="R180" xref="yes"/>
+<pinref part="J6" gate="G$1" pin="4"/>
 </segment>
 </net>
@@
 </segment>
 <segment>
-<pinref part="J4" gate="G$1" pin="8"/>
 <wire x1="353.06" y1="147.32" x2="350.52" y2="147.32" width="0.1524" layer="91"/>
 <label x="350.52" y="147.32" size="1.27" layer="95" font="vector" rot="R180" xref="yes"/>
+<pinref part="J6" gate="G$1" pin="3"/>
 </segment>
 </net>
@@
 </segment>
 <segment>
-<pinref part="J4" gate="G$1" pin="9"/>
 <wire x1="353.06" y1="149.86" x2="350.52" y2="149.86" width="0.1524" layer="91"/>
 <label x="350.52" y="149.86" size="1.27" layer="95" font="vector" rot="R180" xref="yes"/>
+<pinref part="J6" gate="G$1" pin="2"/>
 </segment>
 </net>
@@
 <pinref part="GND40" gate="1" pin="GND"/>
 <wire x1="335.28" y1="127" x2="335.28" y2="132.08" width="0.1524" layer="91"/>
-<pinref part="J4" gate="G$1" pin="2"/>
 <wire x1="335.28" y1="132.08" x2="353.06" y2="132.08" width="0.1524" layer="91"/>
+<pinref part="J6" gate="G$1" pin="9"/>
 </segment>
 <segment>
@@
 <pinref part="P+6" gate="G$1" pin="3V3"/>
 <wire x1="335.28" y1="154.94" x2="335.28" y2="142.24" width="0.1524" layer="91"/>
-<pinref part="J4" gate="G$1" pin="6"/>
 <wire x1="335.28" y1="142.24" x2="353.06" y2="142.24" width="0.1524" layer="91"/>
+<pinref part="J6" gate="G$1" pin="5"/>
 </segment>
 <segment>
@@
 </segment>
 <segment>
-<pinref part="J4" gate="G$1" pin="3"/>
 <wire x1="353.06" y1="134.62" x2="350.52" y2="134.62" width="0.1524" layer="91"/>
 <label x="350.52" y="134.62" size="1.27" layer="95" font="vector" rot="R180" xref="yes"/>
+<pinref part="J6" gate="G$1" pin="8"/>
 </segment>
 <segment>
@@
 </segment>
 <segment>
-<pinref part="J4" gate="G$1" pin="4"/>
 <wire x1="353.06" y1="137.16" x2="350.52" y2="137.16" width="0.1524" layer="91"/>
 <label x="350.52" y="137.16" size="1.27" layer="95" font="vector" rot="R180" xref="yes"/>
+<pinref part="J6" gate="G$1" pin="7"/>
 </segment>
 <segment>
@@
 <pinref part="P+5" gate="VCC" pin="VBAT"/>
 <wire x1="345.44" y1="154.94" x2="345.44" y2="152.4" width="0.1524" layer="91"/>
-<pinref part="J4" gate="G$1" pin="10"/>
 <wire x1="345.44" y1="152.4" x2="353.06" y2="152.4" width="0.1524" layer="91"/>
+<pinref part="J6" gate="G$1" pin="1"/>
 </segment>
 <segment>
@@
 <pinref part="GND41" gate="1" pin="BAT_GND"/>
 <wire x1="345.44" y1="127" x2="345.44" y2="129.54" width="0.1524" layer="91"/>
-<pinref part="J4" gate="G$1" pin="1"/>
 <wire x1="345.44" y1="129.54" x2="353.06" y2="129.54" width="0.1524" layer="91"/>
-</segment>
-<segment>
+<pinref part="J6" gate="G$1" pin="10"/>
+</segment>
+<segment>
