File: hardware/quadcopter.sch (EAGLE design)
At the start: 96 parts, among them J1 AVR_SPI_PRG_6NS, J2 HEADER-0.1IN-2POS-MALE, J3 FTDI_BASICPTH, J5 HEADER-4POS-0.1IN-FEMALE, Q1 MOSFET-VISHAY-SOT23-N-MOSFET, Q2 MOSFET-VISHAY-SOT23-N-MOSFET, Q3 MOSFET-VISHAY-SOT23-N-MOSFET, Q4 MOSFET-VISHAY-SOT23-N-MOSFET, Q5 MOSFET-VISHAY-SOT23-N-MOSFET, U1 ATMEGA128RFA1, U2 IMU_LSM-ST-LSM9DS1-IMU-LGA, U3 MOTOR_PADS-MOLEX-0530470210, U4 MOTOR_PADS-MOLEX-0530470210, U5 MOTOR_PADS-MOLEX-0530470210, U6 MOTOR_PADS-MOLEX-0530470210, U7 3.3V, U8 NET_BRIDGE-BRIDGE-SMD, Y1 CRYSTAL5X3

Commit message: Add files via upload
Connections:
- net BAT_GND: now also C20.1
- net GND: now also J5.3; no longer C20.2, J5.1
- net SDA: now also J5.1; no longer J5.3
- net VBAT: now also C20.2; no longer C20.1
Other:
- moved on the sheet: C20
Changed lines of the file:
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@@
 <part name="D2" library="LED" deviceset="DIODE-LED-LITEON-C170EKT-RED" device="-LITEON-C170EKT-RED-LED" value="red"/>
 <part name="P+24" library="quadparts_prebuilt" deviceset="3V3" device=""/>
+<part name="GND45" library="quadparts_prebuilt" deviceset="BAT_GND" device=""/>
 </parts>
 <sheets>
@@
 <attribute name="NAME" x="112.014" y="132.461" size="1.778" layer="95"/>
 </instance>
-<instance part="C20" gate="G$1" x="66.04" y="132.08" smashed="yes">
-<attribute name="VALUE" x="62.484" y="129.921" size="1.778" layer="96"/>
-<attribute name="NAME" x="66.548" y="132.461" size="1.778" layer="95"/>
+<instance part="C20" gate="G$1" x="71.12" y="134.62" smashed="yes" rot="R90">
+<attribute name="VALUE" x="73.279" y="131.064" size="1.778" layer="96" rot="R90"/>
+<attribute name="NAME" x="70.739" y="135.128" size="1.778" layer="95" rot="R90"/>
 </instance>
 <instance part="C21" gate="G$1" x="121.92" y="132.08" smashed="yes">
@@
 <attribute name="VALUE" x="111.76" y="149.86" size="1.778" layer="96" rot="R180" align="center"/>
 </instance>
-<instance part="GND37" gate="1" x="66.04" y="116.84" smashed="yes">
-<attribute name="VALUE" x="66.04" y="114.3" size="1.778" layer="96" align="center"/>
+<instance part="GND37" gate="1" x="63.5" y="116.84" smashed="yes">
+<attribute name="VALUE" x="63.5" y="114.3" size="1.778" layer="96" align="center"/>
 </instance>
 <instance part="P+20" gate="VCC" x="86.36" y="116.84" smashed="yes">
@@
 <attribute name="VALUE" x="393.7" y="152.4" size="1.778" layer="96" rot="R180" align="center"/>
 </instance>
-<instance part="GND42" gate="1" x="393.7" y="132.08" smashed="yes">
-<attribute name="VALUE" x="393.7" y="129.54" size="1.778" layer="96" align="center"/>
+<instance part="GND42" gate="1" x="398.78" y="127" smashed="yes">
+<attribute name="VALUE" x="398.78" y="124.46" size="1.778" layer="96" align="center"/>
 </instance>
 <instance part="P+23" gate="VCC" x="236.22" y="-25.4" smashed="yes">
@@
 <instance part="P+24" gate="G$1" x="363.22" y="27.94" smashed="yes">
 <attribute name="VALUE" x="363.22" y="30.48" size="1.778" layer="96" rot="R180" align="center"/>
+</instance>
+<instance part="GND45" gate="1" x="63.5" y="129.54" smashed="yes">
+<attribute name="VALUE" x="63.5" y="127" size="1.778" layer="96" align="center"/>
 </instance>
 </instances>
@@
 </segment>
 <segment>
-<pinref part="C20" gate="G$1" pin="2"/>
-<pinref part="GND37" gate="1" pin="GND"/>
-<wire x1="66.04" y1="127" x2="66.04" y2="121.92" width="0.1524" layer="91"/>
-<pinref part="U8" gate="G$1" pin="P2"/>
-<wire x1="66.04" y1="121.92" x2="66.04" y2="119.38" width="0.1524" layer="91"/>
-<wire x1="60.96" y1="121.92" x2="66.04" y2="121.92" width="0.1524" layer="91"/>
-<junction x="66.04" y="121.92"/>
-</segment>
-<segment>
 <pinref part="GND40" gate="1" pin="GND"/>
 <wire x1="335.28" y1="127" x2="335.28" y2="132.08" width="0.1524" layer="91"/>
@@
 </segment>
 <segment>
-<pinref part="J5" gate="G$1" pin="1"/>
-<wire x1="388.62" y1="137.16" x2="393.7" y2="137.16" width="0.1524" layer="91"/>
-<pinref part="GND42" gate="1" pin="GND"/>
-<wire x1="393.7" y1="137.16" x2="393.7" y2="134.62" width="0.1524" layer="91"/>
-</segment>
-<segment>
 <pinref part="R10" gate="G$1" pin="1"/>
 <wire x1="228.6" y1="-71.12" x2="226.06" y2="-71.12" width="0.1524" layer="91"/>
@@
 <pinref part="GND13" gate="1" pin="GND"/>
 <wire x1="198.12" y1="96.52" x2="198.12" y2="93.98" width="0.1524" layer="91"/>
+</segment>
+<segment>
+<pinref part="J5" gate="G$1" pin="3"/>
+<pinref part="GND42" gate="1" pin="GND"/>
+<wire x1="388.62" y1="142.24" x2="398.78" y2="142.24" width="0.1524" layer="91"/>
+<wire x1="398.78" y1="142.24" x2="398.78" y2="129.54" width="0.1524" layer="91"/>
+</segment>
+<segment>
+<pinref part="U8" gate="G$1" pin="P2"/>
+<wire x1="60.96" y1="121.92" x2="63.5" y2="121.92" width="0.1524" layer="91"/>
+<pinref part="GND37" gate="1" pin="GND"/>
+<wire x1="63.5" y1="121.92" x2="63.5" y2="119.38" width="0.1524" layer="91"/>
 </segment>
 </net>
@@
 </segment>
 <segment>
-<pinref part="J5" gate="G$1" pin="3"/>
-<wire x1="388.62" y1="142.24" x2="391.16" y2="142.24" width="0.1524" layer="91"/>
-<label x="391.16" y="142.24" size="1.27" layer="95" font="vector" xref="yes"/>
+<pinref part="J5" gate="G$1" pin="1"/>
+<wire x1="388.62" y1="137.16" x2="391.16" y2="137.16" width="0.1524" layer="91"/>
+<label x="391.16" y="137.16" size="1.27" layer="95" font="vector" xref="yes"/>
 </segment>
 </net>
@@
 <wire x1="50.8" y1="139.7" x2="50.8" y2="142.24" width="0.1524" layer="91"/>
 <pinref part="U7" gate="G$1" pin="IN"/>
-<pinref part="C20" gate="G$1" pin="1"/>
-<wire x1="66.04" y1="134.62" x2="81.28" y2="134.62" width="0.1524" layer="91"/>
-<wire x1="81.28" y1="134.62" x2="81.28" y2="137.16" width="0.1524" layer="91"/>
 <wire x1="81.28" y1="137.16" x2="81.28" y2="139.7" width="0.1524" layer="91"/>
-<junction x="81.28" y="137.16"/>
 <wire x1="81.28" y1="139.7" x2="55.88" y2="139.7" width="0.1524" layer="91"/>
 <junction x="55.88" y="139.7"/>
+<pinref part="C20" gate="G$1" pin="2"/>
+<wire x1="76.2" y1="134.62" x2="81.28" y2="134.62" width="0.1524" layer="91"/>
+<wire x1="81.28" y1="134.62" x2="81.28" y2="137.16" width="0.1524" layer="91"/>
+<junction x="81.28" y="137.16"/>
 </segment>
 <segment>
@@
 <wire x1="236.22" y1="-63.5" x2="236.22" y2="-73.66" width="0.1524" layer="91"/>
 </segment>
-</net>
+<segment>
+<pinref part="GND45" gate="1" pin="BAT_GND"/>
+<wire x1="63.5" y1="132.08" x2="63.5" y2="134.62" width="0.1524" layer="91"/>
+<pinref part="C20" gate="G$1" pin="1"/>
+<wire x1="63.5" y1="134.62" x2="68.58" y2="134.62" width="0.1524" layer="91"/>
+</segment>
+</net>
