File: hardware/quadcopter.sch (EAGLE design)
At the start: 96 parts, among them J1 AVR_SPI_PRG_6NS, J2 HEADER-0.1IN-2POS-MALE, J3 FTDI_BASICPTH, J5 HEADER-4POS-0.1IN-FEMALE, Q1 MOSFET-VISHAY-SOT23-N-MOSFET, Q2 MOSFET-VISHAY-SOT23-N-MOSFET, Q3 MOSFET-VISHAY-SOT23-N-MOSFET, Q4 MOSFET-VISHAY-SOT23-N-MOSFET, Q5 MOSFET-VISHAY-SOT23-N-MOSFET, U1 ATMEGA128RFA1, U2 IMU_LSM-ST-LSM9DS1-IMU-LGA, U3 MOTOR_PADS-MOLEX-0530470210, U4 MOTOR_PADS-MOLEX-0530470210, U5 MOTOR_PADS-MOLEX-0530470210, U6 MOTOR_PADS-MOLEX-0530470210, U7 3.3V, U8 NET_BRIDGE-BRIDGE-SMD, Y1 CRYSTAL5X3

Commit message: Add files via upload
Parts:
- added C22: 0.1uF, quadparts_prebuilt:CAPACITOR-NP_SMD-2012-0805_CERAMIC-0.1UF
- added J6, J7: HEADER-0.1IN-2POS-FEMALE, quadparts_prebuilt:HEADER-0.1IN-2POS-FEMALE
- added Q6: MOSFET-VISHAY-SOT23-N-MOSFET, custom:MOSFET-VISHAY-SOT23-N-MOSFET
- added R29: 10K, quadparts_prebuilt:RESISTOR_SMD-2012-0805-10K
Connections:
- new net 34: Q6.G, R29.2, U1.PB6(OC1B/PCINT6)
- new net N$19: C22.1, J6.2
- new net N$39: D13.C, D14.C, D15.C, D16.C, D18.C, D21.C, D23.C, D25.C, Q6.D
- net BAT_GND: now also Q6.S
- net GND: now also J6.1, R29.1
- net N$38: no longer D13.C, D14.C, D15.C, D16.C, D18.C, D21.C, D23.C, D25.C
- net RESET: now also C22.2
- net RX0: now also J7.1
- net TX0: now also J7.2
Other:
- note added: "FTDI CONNECTOR"
- note added: "LED CONNECTIONS"
- note removed: "LED CONNECTTIONS"
- moved on the sheet: D13, D14, D15, D16, D17, D18, D20, D21, D22, D23, D24, D25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

Commit message: Add files via upload
Parts:
- C12: value 0.01uF -> 10uF; device quadparts_prebuilt:CAPACITOR-NP_SMD-2012-0805_CERAMIC-0.01UF -> quadparts_prebuilt:CAPACITOR-NP_SMD-2012-0805_CERAMIC-10UF
