File: hardware/quadcopter.brd (EAGLE design)
At the start: 130.4 x 130.4 mm, 103 parts, among them J1 AVR_SPI_PRG_6NS, J2 HEADER-0.1IN-2POS-MALE, J3 FTDI_BASICPTH, J5 HEADER-4POS-0.1IN-FEMALE, J6 HEADER-0.1IN-2POS-FEMALE, J7 HEADER-0.1IN-2POS-FEMALE, Q1 MOSFET-VISHAY-SOT23-N-MOSFET, Q2 MOSFET-VISHAY-SOT23-N-MOSFET, Q3 MOSFET-VISHAY-SOT23-N-MOSFET, Q4 MOSFET-VISHAY-SOT23-N-MOSFET, Q5 MOSFET-VISHAY-SOT23-N-MOSFET, Q6 MOSFET-VISHAY-SOT23-N-MOSFET, U1 ATMEGA128RFA1, U2 IMU_LSM-ST-LSM9DS1-IMU-LGA, U3 MOTOR_PADS-MOLEX-0530470210, U4 MOTOR_PADS-MOLEX-0530470210, U5 MOTOR_PADS-MOLEX-0530470210, U6 MOTOR_PADS-MOLEX-0530470210, U7 3.3V, U8 NET_BRIDGE-BRIDGE-SMD, Y1 CRYSTAL5X3

Commit message: Add files via upload
Parts:
- renumbered U$1 to E$1
Changed lines of the file:
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@@
 <attribute name="NAME" x="29" y="26" size="0.9" layer="25" font="vector"/>
 </element>
-<element name="U$1" library="Logos" package="LEBRON_JAMES" value="" x="-19" y="29" smashed="yes"/>
 <element name="U$2" library="quadparts_prebuilt" package="LAYER_LABELS" value="" x="51" y="12" smashed="yes"/>
+<element name="E$1" library="Logos" package="LEBRON_JAMES" value="" x="-19" y="29" smashed="yes"/>
 </elements>
 <signals>

Commit message: Add files via upload
Parts:
- C12: value 0.01uF -> 10uF
- moved C12 5.83 mm to (-5.00, 5.00)
- moved R4 5.00 mm to (8.00, 5.00)
- moved R5 5.00 mm to (11.0, 5.00)
- moved U7 5.00 mm to (11.0, -17.0)
- moved C20 4.00 mm to (15.0, -17.0)
- moved C1 3.00 mm to (-9.00, 19.0)
- moved C2 3.00 mm to (-9.00, 14.0)
- moved C7 3.00 mm to (-12.0, 19.0)
- moved C8 3.00 mm to (-12.0, 14.0)
- renumbered E$1 to U$1
Routing:
- net SDA: track 70.2 -> 116.0 mm, vias 3 -> 2
- net RESET: track 79.8 -> 109.1 mm, vias 2 -> 0
- net 4: track 74.9 -> 100.5 mm, vias 3 -> 0
- net SCL: track 69.5 -> 89.0 mm, vias 3 -> 4
- net GND: track 57.4 -> 74.6 mm, vias 26 -> 41
- net 34: track 54.3 -> 43.3 mm, vias 0 -> 2
- net 9: track 60.6 -> 69.1 mm, vias 4 -> 2
- net N$8: track 16.3 -> 24.8 mm
- net N$39: track 138.0 -> 130.2 mm
- net 8: track 78.8 -> 71.1 mm, vias 1 -> 3
- net N$25: track 12.3 -> 5.05 mm
- net 3: track 78.6 -> 85.2 mm, vias 1 -> 0
- net VBAT: track 57.4 -> 51.4 mm
- net N$19: track 32.6 -> 26.7 mm, vias 0 -> 1
- net MISO: track 36.1 -> 30.3 mm
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- added copper zone on layer 15, net LAYER15_CUTOUT
- added copper zone on layer 2, net LAYER2_CUTOUT

Commit message: Add files via upload
Parts:
- moved C12 3.00 mm to (-5.00, 2.00)
- moved C11 2.00 mm to (-5.00, -2.00)
- moved C14 1.00 mm to (-12.0, -2.00)
Routing:
- net SDA: track 116.0 -> 63.2 mm, vias 2 -> 1
- net 5: track 83.1 -> 113.5 mm, vias 4 -> 1
- net PG1: track 34.4 -> 52.3 mm
- net N$37: track 9.81 -> 27.2 mm
- net N$33: track 9.81 -> 27.2 mm
- net RESET: track 109.1 -> 92.4 mm, vias 0 -> 2
- net 9: track 69.1 -> 85.6 mm
- net 3: track 85.2 -> 70.7 mm, vias 0 -> 2
- net N$38: track 139.0 -> 153.3 mm
- net BAT_GND: track 23.0 -> 36.5 mm, vias 11 -> 10
- net 4: track 100.5 -> 90.4 mm, vias 0 -> 3
- net MISO: track 30.3 -> 40.3 mm
- net 3V3: track 53.4 -> 60.9 mm
- net 8: track 71.1 -> 78.2 mm, vias 3 -> 2
- net TX0: track 65.4 -> 72.3 mm, vias 1 -> 2
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
Commit message: Add files via upload
Routing:
- net PG1: track 52.3 -> 41.3 mm
- net 9: track 85.6 -> 84.4 mm
Changed lines of the file:
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@@
 <setting verticaltext="up"/>
 </settings>
-<grid distance="1" unitdist="mm" unit="mm" style="lines" multiple="1" display="yes" altdistance="5" altunitdist="mil" altunit="mil"/>
+<grid distance="0.1" unitdist="mm" unit="mm" style="lines" multiple="1" display="yes" altdistance="5" altunitdist="mil" altunit="mil"/>
 <layers>
 <layer number="1" name="Top" color="4" fill="1" visible="yes" active="yes"/>
@@
 <wire x1="-28" y1="-29" x2="-27.95" y2="-29.15" width="0.127" layer="1"/>
 <wire x1="-0.25" y1="15" x2="-0.25" y2="11.119" width="0.127" layer="1"/>
-<wire x1="-6" y1="20.75" x2="-0.25" y2="15" width="0.127" layer="16"/>
-<wire x1="-8.25" y1="23" x2="-6" y2="20.75" width="0.127" layer="1"/>
-<wire x1="-24" y1="23" x2="-8.25" y2="23" width="0.127" layer="1"/>
-<wire x1="-24" y1="19.75" x2="-24" y2="23" width="0.127" layer="1"/>
+<wire x1="-9.75" y1="15" x2="-0.25" y2="15" width="0.127" layer="16"/>
+<wire x1="-9.75" y1="15" x2="-16.9" y2="22.15" width="0.127" layer="16"/>
+<wire x1="-16.9" y1="22.1" x2="-16.9" y2="22.15" width="0.127" layer="1"/>
+<wire x1="-24" y1="22.1" x2="-16.9" y2="22.1" width="0.127" layer="1"/>
+<wire x1="-24" y1="19.75" x2="-24" y2="22.1" width="0.127" layer="1"/>
 <wire x1="-27.75" y1="16" x2="-24" y2="19.75" width="0.127" layer="1"/>
 <wire x1="-27.75" y1="-20.75" x2="-27.75" y2="16" width="0.127" layer="1"/>
@@
 <wire x1="-28" y1="-21" x2="-28" y2="-21.045" width="0.127" layer="1"/>
 <via x="-0.25" y="15" extent="1-16" drill="0.2"/>
-<via x="-6" y="20.75" extent="1-16" drill="0.2"/>
+<via x="-16.9" y="22.15" extent="1-16" drill="0.2"/>
 </signal>
 <signal name="8">
@@
 <wire x1="7.5" y1="11.75" x2="12" y2="7.25" width="0.127" layer="1"/>
 <wire x1="4.5" y1="11.75" x2="7.5" y2="11.75" width="0.127" layer="1"/>
-<wire x1="-3.25" y1="19.5" x2="4.5" y2="11.75" width="0.127" layer="2"/>
-<wire x1="-2.75" y1="20" x2="-3.25" y2="19.5" width="0.127" layer="1"/>
-<wire x1="-2.75" y1="20.881" x2="-2.75" y2="20" width="0.127" layer="1"/>
+<wire x1="4.5" y1="11.95" x2="4.5" y2="11.75" width="0.127" layer="2"/>
+<wire x1="4.5" y1="11.95" x2="-2.75" y2="19.2" width="0.127" layer="2"/>
+<wire x1="-2.75" y1="20.881" x2="-2.75" y2="19.2" width="0.127" layer="1"/>
 <wire x1="14" y1="1" x2="14" y2="0.955" width="0.127" layer="1"/>
 <via x="4.5" y="11.75" extent="1-16" drill="0.2"/>
-<via x="-3.25" y="19.5" extent="1-16" drill="0.2"/>
+<via x="-2.75" y="19.2" extent="1-16" drill="0.2"/>
 </signal>
 <signal name="PG1">
@@
 <wire x1="14.5" y1="19" x2="15.5" y2="18" width="0.127" layer="1"/>
 <wire x1="13.5" y1="19" x2="14.5" y2="19" width="0.127" layer="1"/>
-<wire x1="4.5" y1="28" x2="13.5" y2="19" width="0.127" layer="1"/>
-<wire x1="0" y1="28" x2="4.5" y2="28" width="0.127" layer="1"/>
-<wire x1="0" y1="28.25" x2="0" y2="28" width="0.127" layer="1"/>
-<wire x1="-0.25" y1="28.5" x2="0" y2="28.25" width="0.127" layer="16"/>
-<wire x1="-2" y1="28.5" x2="-0.25" y2="28.5" width="0.127" layer="16"/>
-<wire x1="-4" y1="26.5" x2="-2" y2="28.5" width="0.127" layer="1"/>
-<wire x1="-4" y1="23.5" x2="-4" y2="26.5" width="0.127" layer="1"/>
-<wire x1="-4.75" y1="22.75" x2="-4" y2="23.5" width="0.127" layer="1"/>
-<wire x1="-6" y1="22.75" x2="-4.75" y2="22.75" width="0.127" layer="1"/>
-<wire x1="-6" y1="22.25" x2="-6" y2="22.75" width="0.127" layer="1"/>
-<wire x1="-5.75" y1="22" x2="-6" y2="22.25" width="0.127" layer="1"/>
-<wire x1="-3.25" y1="22" x2="-5.75" y2="22" width="0.127" layer="1"/>
-<wire x1="-3.25" y1="20.881" x2="-3.25" y2="22" width="0.127" layer="1"/>
+<wire x1="10.9" y1="21.6" x2="13.5" y2="19" width="0.127" layer="1"/>
+<wire x1="10.9" y1="21.45" x2="10.9" y2="21.6" width="0.127" layer="1"/>
+<wire x1="10.9" y1="21.45" x2="8.15" y2="18.7" width="0.127" layer="16"/>
+<wire x1="-3.2" y1="18.7" x2="8.15" y2="18.7" width="0.127" layer="16"/>
 <wire x1="17" y1="1" x2="17" y2="0.955" width="0.127" layer="1"/>
-<via x="0" y="28.25" extent="1-16" drill="0.2"/>
-<via x="-2" y="28.5" extent="1-16" drill="0.2"/>
+<via x="10.9" y="21.45" extent="1-16" drill="0.2"/>
+<via x="-3.2" y="18.7" extent="1-16" drill="0.2"/>
+<wire x1="-3.25" y1="20.881" x2="-3.25" y2="18.75" width="0.254" layer="1"/>
+<wire x1="-3.25" y1="18.75" x2="-3.2" y2="18.7" width="0.254" layer="1"/>
 </signal>
 <signal name="GND" class="2">

Commit message: Add files via upload
Parts:
- turned C11 to 270 degrees
- turned C2 to 270 degrees
Routing:
- net 5: track 113.5 -> 80.1 mm, vias 1 -> 2
- net 3V3: track 60.9 -> 87.6 mm, vias 23 -> 14
- net 9: track 84.4 -> 59.8 mm
- net SCL: track 95.1 -> 74.7 mm, vias 2 -> 3
- net N$37: track 27.2 -> 12.1 mm
- net N$33: track 27.2 -> 12.1 mm
- net BAT_GND: track 36.5 -> 23.1 mm, vias 10 -> 11
- net RESET: track 92.4 -> 80.6 mm
- net 4: track 90.4 -> 79.6 mm, vias 3 -> 2
- net PG1: track 41.3 -> 30.7 mm
- net N$38: track 153.3 -> 143.5 mm, vias 3 -> 6
- net MISO: track 40.3 -> 30.5 mm
- net SDA: track 63.2 -> 71.5 mm, vias 1 -> 3
- net 3: track 70.7 -> 78.0 mm, vias 2 -> 1
- net SCK: track 41.5 -> 35.1 mm
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